File: wm_1.brd (EAGLE design)
At the start: 110.3 x 34 mm, 22 parts, among them T1 MMBT3904, T2 BT138-V, X1 22-23-2031

Commit message: wip
Parts:
- moved R3 3.13 mm to (30.4, 8.38), turned to 180 degrees
- moved R2 2.56 mm to (18.5, 19.9), turned to 0 degrees
- moved R1 2.28 mm to (18.4, 8.38), turned to 0 degrees
- moved D1 1.98 mm to (33.7, 14.2)
Routing:
- net N$4: track 12.1 -> 3.90 mm
- net N$9: track 20.4 -> 13.6 mm
- net GROUND: track 111.6 -> 107.7 mm
- net N$3: track 16.2 -> 14.3 mm
- net N$5: track 47.1 -> 47.9 mm
- net N$1: track 8.19 -> 8.70 mm
Changed lines of the file:
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@@
 <attribute name="VALUE" x="41.057" y="16.011" size="1.27" layer="27" rot="R270"/>
 </element>
-<element name="D1" library="microbuilder" package="SOD-123" value="1N4148" x="33.972" y="12.256" smashed="yes">
-<attribute name="NAME" x="33.2735" y="13.399" size="0.8128" layer="25" ratio="18"/>
-<attribute name="VALUE" x="33.337" y="10.859" size="0.4064" layer="27" ratio="10"/>
+<element name="D1" library="microbuilder" package="SOD-123" value="1N4148" x="33.718" y="14.2245" smashed="yes">
+<attribute name="NAME" x="33.0195" y="15.3675" size="0.8128" layer="25" ratio="18"/>
+<attribute name="VALUE" x="33.083" y="12.8275" size="0.4064" layer="27" ratio="10"/>
 </element>
 <element name="OK1" library="optocoupler" library_urn="urn:adsk.eagle:library:320" package="DIL6-SMD" package3d_urn="urn:adsk.eagle:package:21970/1" value="4N35SM" x="57.722" y="15.748" smashed="yes" rot="R270">
@@
 <attribute name="VALUE" x="57.087" y="19.558" size="1.27" layer="27" ratio="10" rot="R270"/>
 </element>
-<element name="R1" library="microbuilder" package="1206" value="220k" x="16.2555" y="7.4935" smashed="yes" rot="R90">
-<attribute name="NAME" x="18.478" y="5.9695" size="0.8128" layer="25" ratio="18" rot="R90"/>
-<attribute name="VALUE" x="18.2875" y="8.5095" size="0.4064" layer="27" ratio="10" rot="R90"/>
-</element>
-<element name="R2" library="microbuilder" package="1206" value="220k" x="16.2555" y="21.0185" smashed="yes" rot="R270">
-<attribute name="NAME" x="17.843" y="22.225" size="0.8128" layer="25" ratio="18" rot="R270"/>
-<attribute name="VALUE" x="17.843" y="19.812" size="0.4064" layer="27" ratio="10" rot="R270"/>
-</element>
-<element name="R3" library="microbuilder" package="1206" value="22k" x="33.528" y="8.001" smashed="yes">
-<attribute name="NAME" x="33.3375" y="9.4615" size="0.8128" layer="25" ratio="18"/>
-<attribute name="VALUE" x="33.2105" y="6.1595" size="0.4064" layer="27" ratio="10"/>
+<element name="R1" library="microbuilder" package="1206" value="220k" x="18.352" y="8.3825" smashed="yes">
+<attribute name="NAME" x="16.828" y="6.16" size="0.8128" layer="25" ratio="18"/>
+<attribute name="VALUE" x="19.368" y="6.3505" size="0.4064" layer="27" ratio="10"/>
+</element>
+<element name="R2" library="microbuilder" package="1206" value="220k" x="18.542" y="19.875" smashed="yes">
+<attribute name="NAME" x="17.3355" y="21.4625" size="0.8128" layer="25" ratio="18"/>
+<attribute name="VALUE" x="19.7485" y="21.4625" size="0.4064" layer="27" ratio="10"/>
+</element>
+<element name="R3" library="microbuilder" package="1206" value="22k" x="30.4165" y="8.382" smashed="yes" rot="R180">
+<attribute name="NAME" x="30.607" y="6.9215" size="0.8128" layer="25" ratio="18" rot="R180"/>
+<attribute name="VALUE" x="30.734" y="10.2235" size="0.4064" layer="27" ratio="10" rot="R180"/>
 </element>
 <element name="R4" library="microbuilder" package="1206" value="1k" x="54.674" y="7.938" smashed="yes" rot="R180">
@@
 <wire x1="19.87475" y1="11.6205" x2="19.87475" y2="11.55625" width="0.3048" layer="1"/>
 <wire x1="19.87475" y1="11.4935" x2="19.87475" y2="11.55625" width="0.8128" layer="1"/>
-<wire x1="16.256" y1="11.4935" x2="19.87475" y2="11.4935" width="0.508" layer="1"/>
+<wire x1="16.256" y1="11.4935" x2="19.752" y2="11.4935" width="0.508" layer="1"/>
 <wire x1="16.256" y1="13.147" x2="16.256" y2="11.4935" width="0.508" layer="1"/>
-<wire x1="16.2555" y1="8.8935" x2="16.2555" y2="11.4935" width="0.508" layer="1"/>
 <wire x1="16.2555" y1="11.4935" x2="16.256" y2="11.4935" width="0.508" layer="1"/>
+<wire x1="19.752" y1="8.3825" x2="19.752" y2="11.4935" width="0.508" layer="1"/>
+<wire x1="19.752" y1="11.4935" x2="19.87475" y2="11.4935" width="0.508" layer="1"/>
 </signal>
 <signal name="N$2">
@@
 <wire x1="19.884" y1="16.7005" x2="19.884" y2="16.647" width="0.3048" layer="1"/>
 <wire x1="16.256" y1="16.7005" x2="19.8305" y2="16.7005" width="0.508" layer="1"/>
-<wire x1="16.256" y1="15.047" x2="16.256" y2="16.0655" width="0.508" layer="1"/>
-<wire x1="16.256" y1="16.0655" x2="16.256" y2="16.7005" width="0.508" layer="1"/>
-<wire x1="16.2555" y1="19.6185" x2="16.256" y2="19.6185" width="0.508" layer="1"/>
-<wire x1="16.256" y1="19.6185" x2="16.256" y2="16.7005" width="0.508" layer="1"/>
+<wire x1="16.256" y1="15.047" x2="16.256" y2="16.7005" width="0.508" layer="1"/>
+<wire x1="19.942" y1="19.875" x2="19.942" y2="16.647" width="0.508" layer="1"/>
+<wire x1="19.942" y1="16.647" x2="19.884" y2="16.647" width="0.508" layer="1"/>
 </signal>
 <signal name="N$3">
@@
 <wire x1="44.4705" y1="16.7865" x2="43.942" y2="16.786" width="0.3048" layer="1"/>
 <wire x1="34.034" y1="16.616" x2="33.981" y2="16.564" width="0.3048" layer="1"/>
-<wire x1="34.034" y1="16.616" x2="35.8225" y2="16.6165" width="0.508" layer="1"/>
+<wire x1="34.034" y1="16.616" x2="35.441346875" y2="16.61639375" width="0.508" layer="1"/>
+<wire x1="35.441346875" y1="16.61639375" x2="35.568275" y2="16.616428125" width="0.508" layer="1"/>
+<wire x1="35.568275" y1="16.616428125" x2="35.8225" y2="16.6165" width="0.508" layer="1"/>
 <wire x1="35.8225" y1="16.6165" x2="44.7675" y2="16.6165" width="0.508" layer="1"/>
 <wire x1="44.7675" y1="16.6165" x2="44.7675" y2="16.4895" width="0.508" layer="1"/>
-<wire x1="35.822" y1="12.256" x2="35.8225" y2="16.6165" width="0.508" layer="1"/>
+<wire x1="35.568" y1="14.2245" x2="35.568275" y2="16.616428125" width="0.508" layer="1"/>
 </signal>
 <signal name="N$4">
@@
 <contactref element="D1" pad="C"/>
 <contactref element="T1" pad="B"/>
-<wire x1="32.128" y1="12.2555" x2="32.122" y2="12.256" width="0.3048" layer="1"/>
+<wire x1="31.874" y1="14.224" x2="31.868" y2="14.2245" width="0.3048" layer="1"/>
 <wire x1="28.884" y1="16.8705" x2="28.884" y2="16.647" width="0.3048" layer="1"/>
 <wire x1="28.884" y1="16.647" x2="28.884" y2="16.6165" width="0.508" layer="1"/>
 <wire x1="28.884" y1="16.6165" x2="32.134" y2="16.616" width="0.508" layer="1"/>
-<wire x1="32.134" y1="16.616" x2="32.1335" y2="12.2555" width="0.508" layer="1"/>
-<wire x1="32.1335" y1="12.2555" x2="32.122" y2="12.256" width="0.508" layer="1"/>
-<wire x1="32.122" y1="12.256" x2="32.1225" y2="8.001" width="0.508" layer="1"/>
-<wire x1="32.1225" y1="8.001" x2="32.128" y2="8.001" width="0.508" layer="1"/>
+<wire x1="32.26065" y1="14.207428125" x2="31.868" y2="14.2245" width="0.508" layer="1"/>
+<wire x1="32.26065" y1="14.207428125" x2="32.134" y2="16.616" width="0" layer="19" extent="1-1"/>
+<wire x1="31.8165" y1="8.382" x2="31.868" y2="14.2245" width="0" layer="19" extent="1-1"/>
 </signal>
 <signal name="N$5">
@@
 <contactref element="R4" pad="2"/>
 <contactref element="C1" pad="+"/>
-<wire x1="34.928" y1="8.0645" x2="34.928" y2="8.001" width="0.3048" layer="1"/>
 <wire x1="43.942" y1="8.128" x2="43.942" y2="8.486" width="0.3048" layer="1"/>
 <wire x1="43.942" y1="8.4455" x2="43.942" y2="8.486" width="0.1524" layer="1"/>
@@
 <wire x1="44.663" y1="8.4865" x2="43.942" y2="8.486" width="0.1524" layer="1"/>
 <wire x1="28.884" y1="11.547" x2="25.654" y2="11.547" width="0.508" layer="1"/>
-<wire x1="25.654" y1="5.2705" x2="25.654" y2="11.547" width="0.508" layer="1"/>
-<wire x1="34.928" y1="5.2705" x2="44.0055" y2="5.2705" width="0.508" layer="1"/>
+<wire x1="25.654" y1="5.2705" x2="25.654" y2="8.1915" width="0.508" layer="1"/>
+<wire x1="25.654" y1="8.1915" x2="25.654" y2="11.547" width="0.508" layer="1"/>
 <wire x1="44.0055" y1="5.2705" x2="53.2735" y2="5.2705" width="0.508" layer="1"/>
-<wire x1="34.928" y1="5.2705" x2="25.654" y2="5.2705" width="0.508" layer="1"/>
-<wire x1="34.928" y1="8.001" x2="34.928" y2="5.2705" width="0.508" layer="1"/>
+<wire x1="44.0055" y1="5.2705" x2="25.654" y2="5.2705" width="0.508" layer="1"/>
 <wire x1="53.274" y1="7.938" x2="53.2735" y2="5.2705" width="0.508" layer="1"/>
 <wire x1="43.942" y1="8.486" x2="43.942" y2="5.334" width="0.508" layer="1"/>
 <wire x1="43.942" y1="5.334" x2="44.0055" y2="5.2705" width="0.508" layer="1"/>
+<wire x1="29.0165" y1="8.382" x2="29.0165" y2="8.1915" width="0.508" layer="1"/>
+<wire x1="29.0165" y1="8.1915" x2="25.654" y2="8.1915" width="0.508" layer="1"/>
 </signal>
 <signal name="N$6">
@@
 <wire x1="14.478" y1="2.159" x2="16.1925" y2="2.159" width="2.286" layer="1"/>
 <wire x1="16.1925" y1="2.159" x2="96.7105" y2="2.159" width="2.286" layer="1"/>
-<wire x1="16.2555" y1="6.0935" x2="16.2555" y2="2.159" width="0.508" layer="1"/>
 <wire x1="16.2555" y1="2.159" x2="16.1925" y2="2.159" width="0.508" layer="1"/>
+<wire x1="16.1925" y1="2.159" x2="16.952" y2="8.3825" width="0" layer="19" extent="1-1"/>
 </signal>
 <signal name="GND">
@@
 <wire x1="7.2775" y1="16.5951" x2="7.2775" y2="19.8505" width="2.286" layer="1"/>
 <wire x1="7.2775" y1="19.8505" x2="14.605" y2="27.178" width="2.286" layer="1"/>
-<wire x1="16.2555" y1="27.178" x2="16.2555" y2="22.4185" width="0.508" layer="1"/>
-<wire x1="14.2245" y1="27.242" x2="16.1915" y2="27.242" width="0.508" layer="1"/>
-<wire x1="16.1915" y1="27.242" x2="16.2555" y2="27.178" width="0.508" layer="1"/>
 <wire x1="14.605" y1="27.178" x2="14.2245" y2="27.242" width="0" layer="19" extent="1-1"/>
+<wire x1="17.142" y1="19.875" x2="14.605" y2="27.178" width="0" layer="19" extent="1-1"/>
 </signal>
 <signal name="ZERO">

Commit message: v2.1
Parts:
- removed C4: 0.05, rcl:C1206
- removed F1: (no value), fuse:GSH15
- added F2: (no value), fuse:SH22,5A
- C1: value 10uF 10V -> 10 uF 10V; device rcl:140CLH-1010 -> rcl:C1206
- C2: device rcl:C0805 -> rcl:C1206
- R6: value 470 -> 330
- R7: value 360 -> 380
- R8: value 1k -> 470
- moved X1 45.4 mm to (51.4, 9.14), turned to 0 degrees
- moved OUT 42.9 mm to (63.1, 9.46)
- moved R8 42.0 mm to (49.8, 14.9)
- moved R7 39.9 mm to (38.5, 28.2)
- moved OK2 35.0 mm to (51.1, 23.7), turned to 0 degrees
- moved C3 33.6 mm to (41.4, 22.9)
- moved R5 33.3 mm to (35.5, 22.9)
- moved R4 22.9 mm to (31.8, 8.13)
- moved R6 18.4 mm to (57.9, 26.9), turned to 90 degrees
- moved OK1 18.0 mm to (39.8, 14.0)
- moved C1 13.4 mm to (30.5, 13.1), turned to 90 degrees
- moved T2 9.08 mm to (64.0, 28.7)
- moved D1 6.67 mm to (27.2, 12.6), turned to 90 degrees
- moved R3 6.42 mm to (24.0, 8.06)
- moved B1 6.29 mm to (18.1, 14.2)
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Connections:
- removed net N$8: C4.1, R6.2, R7.1
- removed net N$9: F1.2, IN.1, R2.1
- new net FAZA: F2.1, IN.1
- net GATE: now also R6.2
- net HOT: now also F2.2, R2.1, R7.1; no longer F1.1, R6.1
- net LOAD: now also R6.1; no longer C4.2
- net N$3: now also C1.2; no longer C1.-
- net N$5: now also C1.1; no longer C1.+
Routing:
- net GATE: track 136.8 -> 10.1 mm
- net GROUND: track 107.7 -> 71.6 mm
- net GND: track 59.9 -> 26.2 mm
- net ZERO: track 56.4 -> 26.6 mm
- net N$5: track 47.9 -> 19.5 mm
- net N$4: track 3.90 -> 19.2 mm
- net N$9: track 13.6 -> 0.00 mm
- net FAZA: track 0.00 -> 12.8 mm
- net HOT: track 61.5 -> 72.4 mm
- net N$7: track 26.2 -> 17.6 mm
- net N$8: track 7.45 -> 0.00 mm
- net N$3: track 14.3 -> 7.34 mm
- net LOAD: track 49.6 -> 44.3 mm
- net N$16: track 3.80 -> 8.75 mm
- net ON/OFF: track 10.4 -> 5.88 mm
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Other:
- board size 110.3 x 34 mm -> 69.5 x 35 mm

Commit message: v2.2
Parts:
- moved R7 5.22 mm to (35.0, 24.3), turned to 90 degrees
- moved C1 3.45 mm to (28.5, 10.3)
- moved R5 3.38 mm to (38.5, 24.4), turned to 270 degrees
- moved D1 2.54 mm to (26.7, 15.1), turned to 0 degrees
- moved R3 2.37 mm to (24.8, 10.3), turned to 270 degrees
- moved R4 2.13 mm to (32.2, 10.2), turned to 270 degrees
- moved T1 1.68 mm to (26.7, 19.1), turned to 0 degrees
- moved R1 1.62 mm to (15.3, 8.19)
- moved B1 1.60 mm to (16.5, 14.4)
- moved C3 1.55 mm to (42.0, 24.4), turned to 270 degrees
- moved C2 0.46 mm to (9.59, 14.4)
- moved R2 0.14 mm to (15.1, 21.6)
Routing:
- net N$16: track 8.75 -> 16.4 mm
- net N$4: track 19.2 -> 13.1 mm
- net N$5: track 19.5 -> 14.2 mm
- net GROUND: track 71.6 -> 75.1 mm
- net N$6: track 10.4 -> 7.93 mm
- net N$7: track 17.6 -> 20.0 mm
- net HOT: track 72.4 -> 71.0 mm
- net LOAD: track 44.3 -> 43.5 mm
- net N$1: track 10.5 -> 9.76 mm
- net GND: track 26.2 -> 25.6 mm
